File: pcb/aquarius-node-hw.kicad_pcb (KiCad board)
At the start: 4 copper layers, 50 x 50 mm, 275 parts, among them J2 USB_C_USB2.0_16P, Q1 MMBT2222A, SW1 SKRPABE010, SW2 SKRPABE010, U1 ESP32-S3-WROOM-1-N16R2, U2 LM66200DRLR, U3 USBLC6-2P6, U4 MCP23017T-E/ML, U7 AZ1084-3.3

Commit message: admin updates after 3.1
Parts:
- D1: footprint LED_SMD:LED_WS2812B-2020_PLCC4_2.0x2.0mm -> CRGM Passive:LED_WS2812B-2020_PLCC4_2.0x2.0mm
Changed lines of the file:
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@@
 		(sheetname "/MCU/")
 		(sheetfile "mcu.kicad_sch")
+		(units
+			(unit
+				(name "A")
+				(pins "1" "3" "2" "4")
+			)
+		)
 		(attr smd)
 		(duplicate_pad_numbers_are_jumpers no)
@@
 		(embedded_fonts no)
 	)
-	(footprint "LED_SMD:LED_WS2812B-2020_PLCC4_2.0x2.0mm"
+	(footprint "CRGM Passive:LED_WS2812B-2020_PLCC4_2.0x2.0mm"
 		(layer "F.Cu")
 		(at 81.65 75.15 180)
@@
 		(tags "LED RGB NeoPixel Nano PLCC-4 2020")
 		(property "Reference" "D1"
-			(at 0 -2 180)
+			(at -3.35 0.15 180)
 			(layer "F.SilkS")
 			(hide yes)
@@
 			(at 0 2.2 180)
 			(layer "F.Fab")
-			(hide yes)
 			(effects
 				(font
@@
 		(sheetname "/MCU/")
 		(sheetfile "mcu.kicad_sch")
+		(units
+			(unit
+				(name "A")
+				(pins "3" "4" "2" "1")
+			)
+		)
 		(attr smd)
 		(duplicate_pad_numbers_are_jumpers no)
@@
 		)
 		(fp_line
-			(start -1.6 1.15)
-			(end 1.6 1.15)
+			(start -1.3 -1.15)
+			(end 1.6 -1.15)
 			(stroke
 				(width 0.12)
@@
 		)
 		(fp_line
-			(start -1.6 1.15)
-			(end -1.6 -1.15)
+			(start -1.3 -1.15)
+			(end -1.6 -0.85)
 			(stroke
 				(width 0.12)
-				(type solid)
+				(type default)
 			)
 			(layer "F.SilkS")
 		)
 		(fp_line
-			(start -1.6 -1.15)
-			(end 1.6 -1.15)
+			(start -1.6 1.15)
+			(end 1.6 1.15)
 			(stroke
 				(width 0.12)
@@
 			(layer "F.SilkS")
 		)
-		(fp_circle
-			(center -1.606158 -1.14)
-			(end -1.526158 -1.14)
+		(fp_line
+			(start -1.6 1.15)
+			(end -1.6 -0.85)
 			(stroke
-				(width 0.1)
-				(type default)
+				(width 0.12)
+				(type solid)
 			)
-			(fill yes)
 			(layer "F.SilkS")
 		)
 		(fp_line
-			(start 1.52 1.25)
-			(end 1.52 -1.25)
+			(start 1.25 1.05)
+			(end 1.25 -1.05)
 			(stroke
 				(width 0.05)
@@
 		)
 		(fp_line
-			(start 1.52 -1.25)
-			(end -1.52 -1.25)
+			(start 1.25 -1.05)
+			(end -1.3 -1.05)
 			(stroke
 				(width 0.05)
@@
 		)
 		(fp_line
-			(start -1.52 1.25)
-			(end 1.52 1.25)
+			(start -1.3 1.05)
+			(end 1.25 1.05)
 			(stroke
 				(width 0.05)
@@
 		)
 		(fp_line
-			(start -1.52 -1.25)
-			(end -1.52 1.25)
+			(start -1.3 -1.05)
+			(end -1.3 1.05)
 			(stroke
 				(width 0.05)
@@
 		)
 		(fp_text user "${REFERENCE}"
-			(at 0.0175 1.75 180)
+			(at 3.15 -2.2 180)
 			(layer "F.Fab")
 			(effects
@@
 		(sheetname "/Power/")
 		(sheetfile "power.kicad_sch")
+		(units
+			(unit
+				(name "A")
+				(pins "1" "2")
+			)
+		)
 		(attr smd)
 		(duplicate_pad_numbers_are_jumpers no)
@@
 			)
 		)
-		(property "LCSC1" "C190608"
-			(at 0 0 0)
+		(property "Package" ""
+			(at 0 0 180)
 			(unlocked yes)
 			(layer "F.Fab")
@@
 			)
 		)
-		(property "LCSC2" "C94417"
-			(at 0 0 0)
+		(property "Sim.Device" "NPN"
+			(at 0 0 180)
+			(unlocked yes)
+			(layer "F.Fab")
+			(hide yes)
+			(effects
+				(font
+					(size 1 1)
+					(thickness 0.15)
+				)
+			)
+		)
+		(property "Sim.Pins" "1=B 2=E 3=C"
+			(at 0 0 180)
 			(unlocked yes)
 			(layer "F.Fab")
@@
 		(sheetname "/MCU/")
 		(sheetfile "mcu.kicad_sch")
+		(units
+			(unit
+				(name "A")
+				(pins "1" "3" "2")
+			)
+		)
 		(attr smd)
 		(duplicate_pad_numbers_are_jumpers no)
@@
 		(sheetname "/Power/")
 		(sheetfile "power.kicad_sch")
+		(units
+			(unit
+				(name "A")
+				(pins "1" "2")
+			)
+		)
 		(attr smd)
 		(duplicate_pad_numbers_are_jumpers no)
@@
 		(sheetname "/Power/")
 		(sheetfile "power.kicad_sch")
+		(units
+			(unit
+				(name "A")
+				(pins "3" "1" "2")
+			)
+		)
 		(attr smd)
 		(duplicate_pad_numbers_are_jumpers no)
@@
 		(sheetname "/MCU/")
 		(sheetfile "mcu.kicad_sch")
+		(units
+			(unit
+				(name "A")
+				(pins "1" "3" "2" "4")
+			)
+		)
 		(attr smd)
 		(duplicate_pad_numbers_are_jumpers no)
@@
 		(sheetname "/MCU/")
 		(sheetfile "mcu.kicad_sch")
+		(units
+			(unit
+				(name "A")
+				(pins "1" "2")
+			)
+		)
 		(attr smd)
 		(duplicate_pad_numbers_are_jumpers no)
@@
 		(sheetname "/Power/")
 		(sheetfile "power.kicad_sch")
+		(units
+			(unit
+				(name "A")
+				(pins "1" "2")
+			)
+		)
 		(zone_connect 1)
 		(attr exclude_from_bom allow_soldermask_bridges)
@@
 		(sheetname "/Power/")
 		(sheetfile "power.kicad_sch")
+		(units
+			(unit
+				(name "A")
+				(pins "1" "2")
+			)
+		)
 		(zone_connect 1)
 		(attr exclude_from_bom allow_soldermask_bridges)
