File: pcb/mcu.kicad_sch (KiCad schematic)
At the start: 35 parts, among them Q1 MMBT2222A, SW1 SKRPABE010, SW2 SKRPABE010, U1 ESP32-S3-WROOM-1-N16R2

Commit message: admin updates after 3.1
Parts:
- D1: footprint LED_SMD:LED_WS2812B-2020_PLCC4_2.0x2.0mm -> CRGM Passive:LED_WS2812B-2020_PLCC4_2.0x2.0mm
Changed lines of the file:
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@@
 			)
 		)
-		(property "Footprint" "LED_SMD:LED_WS2812B-2020_PLCC4_2.0x2.0mm"
+		(property "Footprint" "CRGM Passive:LED_WS2812B-2020_PLCC4_2.0x2.0mm"
 			(at 233.68 100.33 0)
 			(hide yes)
